File: M302.kicad_pcb (KiCad board)
At the start: 2 copper layers, 68.6 x 53.3 mm, 8 parts, among them P1 Power, P2 Analog, P3 Digital, P4 Digital, P5 CONN_01X01, P6 CONN_01X01, P7 CONN_01X01, P8 CONN_01X01

Commit message: とりあえず
Parts:
- added C1: 100uF/25V, Capacitor_THT:CP_Radial_D5.0mm_P2.00mm, F.Cu at (124.3, 117.5)
- added J1: I2C-1, Connector_JST:JST_XH_B4B-XH-A_1x04_P2.50mm_Vertical, F.Cu at (116.1, 108.6)
- added J2: I2C-2, Connector_JST:JST_XH_B4B-XH-A_1x04_P2.50mm_Vertical, F.Cu at (125.6, 108.6)
- added J3: I2C-3, Connector_JST:JST_XH_B4B-XH-A_1x04_P2.50mm_Vertical, F.Cu at (134.5, 113.0)
- added J4: I2C-4, Connector_JST:JST_XH_B4B-XH-A_1x04_P2.50mm_Vertical, F.Cu at (144.0, 113.0)
- added J5: I2C-D400, Connector_JST:JST_XH_B7B-XH-A_1x07_P2.50mm_Vertical, F.Cu at (138.9, 97.8)
- added J6: W5500, Connector_PinHeader_2.54mm:PinHeader_2x05_P2.54mm_Vertical, F.Cu at (169.4, 104.8)
- added J7: IM920, Connector_JST:JST_XH_B6B-XH-A_1x06_P2.50mm_Vertical, F.Cu at (156.7, 114.9)
- added J8: PWR, Connector_JST:JST_XH_B2B-XH-A_1x02_P2.50mm_Vertical, F.Cu at (115.4, 118.7)
- added J9: VSW, Connector_PinHeader_2.54mm:PinHeader_1x03_P2.54mm_Vertical, F.Cu at (133.2, 118.7)
- added R1: 10k, Resistor_THT:R_Axial_DIN0207_L6.3mm_D2.5mm_P10.16mm_Horizontal, F.Cu at (125.0, 90.2)
- added SW1: CPU_RESET, HOLLY:TVDT18-050, F.Cu at (117.3, 77.5)
- added SW2: D400_RESET, HOLLY:TVDT18-050, F.Cu at (117.3, 85.7)
- added SW3: IM920_RESET, HOLLY:TVDT18-050, F.Cu at (117.3, 94.0)
- added U1: SFE-BOB-12009, HOLLY:SFE-BOB-12009, F.Cu at (153.5, 87.6)
