File: M302.kicad_pcb (KiCad board)
At the start: 2 copper layers, 68.6 x 53.3 mm, 28 parts, among them J1 I2C-SHT3x, J2 I2C-ThmCp, J3 I2C-3, J4 I2C-4, J5 I2C-D400, J6 W5500, J7 IM920, J8 PWR+5V, J9 ANALOG-IN, P1 Power, P2 Analog, P3 Digital, P4 Digital, P5 CONN_01X01, P6 CONN_01X01, P7 CONN_01X01, P8 CONN_01X01, SW1 CPU, SW2 D400, SW3 IM920, U1 SFE-BOB-12009

Commit message: sche: KiCAD 7.0対応
Other:
- net class Default removed
