File: M302.kicad_sch (KiCad schematic)
At the start: 28 parts

Commit message: KiCAD new version
Parts:
- C1, C3: value (none) -> 100uF/25V; footprint (none) -> Capacitor_THT:CP_Radial_D5.0mm_P2.00mm
- C2, C4: value (none) -> 0.1μF; footprint (none) -> Capacitor_THT:C_Disc_D3.0mm_W2.0mm_P2.50mm
- J1: value (none) -> I2C-SHT3x; footprint (none) -> Connector_JST:JST_XH_B4B-XH-A_1x04_P2.50mm_Vertical
- J2: value (none) -> I2C-ThmCp; footprint (none) -> Connector_JST:JST_XH_B4B-XH-A_1x04_P2.50mm_Vertical
- J3: value (none) -> I2C-3; footprint (none) -> Connector_JST:JST_XH_B4B-XH-A_1x04_P2.50mm_Vertical
- J4: value (none) -> I2C-4; footprint (none) -> Connector_JST:JST_XH_B4B-XH-A_1x04_P2.50mm_Vertical
- J5: value (none) -> I2C-D400; footprint (none) -> Connector_JST:JST_XH_B7B-XH-A_1x07_P2.50mm_Vertical
- J6: value (none) -> W5500; footprint (none) -> Connector_PinHeader_2.54mm:PinHeader_2x05_P2.54mm_Vertical
- J7: value (none) -> IM920; footprint (none) -> Connector_JST:JST_XH_B6B-XH-A_1x06_P2.50mm_Vertical
- J8: value (none) -> PWR+5V; footprint (none) -> Connector_JST:JST_XH_B2B-XH-A_1x02_P2.50mm_Vertical
- J9: value (none) -> ANALOG-IN; footprint (none) -> Connector_JST:JST_XH_B8B-XH-A_1x08_P2.50mm_Vertical
- P1: value (none) -> Power; footprint (none) -> Socket_Arduino_Uno:Socket_Strip_Arduino_1x08
- P2: value (none) -> Analog; footprint (none) -> Socket_Arduino_Uno:Socket_Strip_Arduino_1x06
- P3: value (none) -> Digital; footprint (none) -> Socket_Arduino_Uno:Socket_Strip_Arduino_1x10
- P4: value (none) -> Digital; footprint (none) -> Socket_Arduino_Uno:Socket_Strip_Arduino_1x08
- P5, P6, P7, P8: value (none) -> CONN_01X01; footprint (none) -> Socket_Arduino_Uno:Arduino_1pin
- R1, R2, R3: value (none) -> 10k; footprint (none) -> Resistor_THT:R_Axial_DIN0207_L6.3mm_D2.5mm_P7.62mm_Horizontal
- SW1: value (none) -> CPU; footprint (none) -> HOLLY:TVDT18-050
- SW2: value (none) -> D400; footprint (none) -> HOLLY:TVDT18-050
- SW3: value (none) -> IM920; footprint (none) -> HOLLY:TVDT18-050
- U1: value (none) -> SFE-BOB-12009; footprint (none) -> HOLLY:SFE-BOB-12009
Connections:
- net +3.3V: now reaches P1.4 (Pin_4)
- net +3.3V: now also C3.1, C4.1, J6.1 (Pin_1), J7.4 (Pin_4), U1.LV
