File: M302.kicad_sch (KiCad schematic)
At the start: 28 parts, among them J1 I2C-SHT3x, J2 I2C-ThmCp, J3 I2C-3, J4 I2C-4, J5 I2C-D400, J6 W5500, J7 IM920, J8 PWR+5V, J9 ANALOG-IN, P1 Power, P2 Analog, P3 Digital, P4 Digital, P5 CONN_01X01, P6 CONN_01X01, P7 CONN_01X01, P8 CONN_01X01, SW1 CPU, SW2 D400, SW3 IM920, U1 SFE-BOB-12009

Commit message: Lab Support九州 ヴァージョン
Other:
- company: HOLLY&Co.,Ltd. -> LSQ
- title: M302 Measurement Equipment Type Light -> LY9302 Measurement Equipment Type Light
Changed lines of the file:
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@@
 	(paper "A4")
 	(title_block
-		(title "M302 Measurement Equipment Type Light")
-		(date "2022-07-05")
-		(rev "1.12")
-		(company "HOLLY&Co.,Ltd.")
+		(title "LY9302 Measurement Equipment Type Light")
+		(date "2025-01-27")
+		(rev "1.0")
+		(company "LSQ")
 		(comment 1 "Use W5500 I/F for LAN networking")
 		(comment 2 "Use IM920 I/F for Radio connection")
@@
 	(label "A2"
 		(at 132.08 170.18 0)
-		(fields_autoplaced yes)
 		(effects
 			(font
@@
 	(label "6(**)"
 		(at 190.5 111.76 0)
-		(fields_autoplaced yes)
 		(effects
 			(font
@@
 	(label "A3"
 		(at 132.08 175.26 0)
-		(fields_autoplaced yes)
 		(effects
 			(font
@@
 	(label "3(**)"
 		(at 190.5 119.38 0)
-		(fields_autoplaced yes)
 		(effects
 			(font
@@
 	(label "5(**)"
 		(at 190.5 114.3 0)
-		(fields_autoplaced yes)
 		(effects
 			(font
@@
 	(label "12(MISO)"
 		(at 190.5 93.98 0)
-		(fields_autoplaced yes)
 		(effects
 			(font
@@
 	(label "8"
 		(at 190.5 104.14 0)
-		(fields_autoplaced yes)
 		(effects
 			(font
@@
 	(label "Reset"
 		(at 142.24 96.52 0)
-		(fields_autoplaced yes)
 		(effects
 			(font
@@
 	(label "A5(SCL)"
 		(at 190.5 81.28 0)
-		(fields_autoplaced yes)
 		(effects
 			(font
@@
 	(label "1(Tx)"
 		(at 190.5 124.46 0)
-		(fields_autoplaced yes)
 		(effects
 			(font
@@
 	(label "AREF"
 		(at 190.5 86.36 0)
-		(fields_autoplaced yes)
 		(effects
 			(font
@@
 	(label "13(SCK)"
 		(at 190.5 91.44 0)
-		(fields_autoplaced yes)
 		(effects
 			(font
@@
 	(label "2"
 		(at 190.5 121.92 0)
-		(fields_autoplaced yes)
 		(effects
 			(font
@@
 	(label "IOREF"
 		(at 160.02 87.63 90)
-		(fields_autoplaced yes)
 		(effects
 			(font
@@
 	(label "Vin"
 		(at 149.86 87.63 90)
-		(fields_autoplaced yes)
 		(effects
 			(font
@@
 	(label "A0"
 		(at 132.08 160.02 0)
-		(fields_autoplaced yes)
 		(effects
 			(font
@@
 	(label "7"
 		(at 190.5 109.22 0)
-		(fields_autoplaced yes)
 		(effects
 			(font
@@
 	(label "10(**/SS)"
 		(at 190.5 99.06 0)
-		(fields_autoplaced yes)
 		(effects
 			(font
@@
 	(label "0(Rx)"
 		(at 190.5 127 0)
-		(fields_autoplaced yes)
 		(effects
 			(font
@@
 	(label "9(**)"
 		(at 190.5 101.6 0)
-		(fields_autoplaced yes)
 		(effects
 			(font
@@
 	(label "A4(SDA)"
 		(at 190.5 83.82 0)
-		(fields_autoplaced yes)
 		(effects
 			(font
@@
 	(label "A1"
 		(at 132.08 165.1 0)
-		(fields_autoplaced yes)
 		(effects
 			(font
@@
 	(label "4"
 		(at 190.5 116.84 0)
-		(fields_autoplaced yes)
 		(effects
 			(font
@@
 	(label "11(**/MOSI)"
 		(at 190.5 96.52 0)
-		(fields_autoplaced yes)
-		(effects
-			(font
+		(effects
+			(font
